File: hardware/pcb/control_boards/xt_v03/shruthi_control_board_xt_v03.kicad_pcb (KiCad board)
At the start: 2 copper layers, 286 x 99.4 mm, 129 parts, among them IC1 24LC512, IC10 ATMEGA644p, IC2 74HC165N, IC3 74HC165N, IC4 4051, IC5 4051, IC6 4051, IC7 4051, IC8 74595N, IC9 74HC165N, J1 CV, J2 POWER, J3 M03PTH, J4 POWER, Q1 20MHz, SW1 Encoder, U1 AVRISP, X1 MIDI, X2 MIDI

Commit message: fix pin numbering for pot footprint
Connections:
- JP2 pad 1: Net-(R8-E) -> Net-(JP2-Pad1)
- JP2 pad 2: Net-(R8-S) -> Net-(JP2-Pad2)
- JP2 pad 3: Net-(R8-A) -> Net-(JP2-Pad3)
Routing:
- net Net-(R8-A): track 15.4 -> 0.00 mm
- net Net-(JP2-Pad3): track 0.00 -> 15.4 mm
- net Net-(R8-E): track 15.4 -> 0.00 mm
- net Net-(JP2-Pad1): track 0.00 -> 15.4 mm
- net Net-(R8-S): track 14.3 -> 0.00 mm
- net Net-(JP2-Pad2): track 0.00 -> 14.3 mm
